File: rev1.kicad_pcb (KiCad board)
At the start: 2 copper layers, 43.2 x 18.4 mm, 6 parts, among them P1 CONN_01X02, P2 CONN_01X03, P3 CONN_01X01, Q1 AOT240L

Commit message: Added PDF of schematic, and renders of board
Other:
- board text added: "By Dumle29"
- board text added: "VBB switcher"
- board text added: "git.io/voX63"
Changed lines of the file:
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@@
     (links 9)
     (no_connects 1)
-    (area 115.494999 91.999999 158.825001 110.565001)
+    (area 115.494999 89.7518 158.825001 110.8332)
     (thickness 1.6)
-    (drawings 56)
+    (drawings 59)
     (tracks 44)
     (zones 0)
@@
     (visible_elements FFFFFF7F)
     (pcbplotparams
-      (layerselection 0x00030_80000001)
-      (usegerberextensions false)
+      (layerselection 0x010f0_80000001)
+      (usegerberextensions true)
       (excludeedgelayer true)
       (linewidth 0.100000)
@@
       (outputformat 1)
       (mirror false)
-      (drillshape 1)
+      (drillshape 0)
       (scaleselection 1)
-      (outputdirectory ""))
+      (outputdirectory gerbers/))
   )
   (net 0 "")
@@
     )
   )
+  (gr_text "VBB switcher" (at 116.14912 103.04272 360) (layer B.SilkS)
+    (effects (font (size 1.5 1.5) (thickness 0.3)) (justify right mirror))
+  )
+  (gr_text git.io/voX63 (at 116.0272 106.0196 360) (layer B.SilkS)
+    (effects (font (size 1.5 1.5) (thickness 0.3)) (justify right mirror))
+  )
+  (gr_text "By Dumle29" (at 115.951 108.9406 360) (layer B.SilkS)
+    (effects (font (size 1.5 1.5) (thickness 0.3)) (justify right mirror))
+  )
   (gr_line (start 145.415 104.775) (end 145.415 104.521) (layer B.SilkS) (width 0.2))
